File: board/board.kicad_pcb (KiCad board)
At the start: 2 copper layers, 21 x 13 mm, 1 part

Commit message: initial
Parts:
- removed LOGO1: Logo_Open_Hardware_Small, Symbol:OSHW-Symbol_6.7x6mm_SilkScreen
- added C1: 100n, Capacitor_SMD:C_0603_1608Metric, F.Cu at (78.0, 97.8)
- added C10: 1nF, Capacitor_SMD:C_1825_4564Metric, B.Cu at (98.8, 96.7)
- added C2: 1uF, Capacitor_SMD:C_0603_1608Metric, F.Cu at (85.8, 97.8)
- added C3: 2.2uF, Capacitor_SMD:C_1210_3225Metric, F.Cu at (83.0, 90.6)
- added C4: 10uF, Capacitor_SMD:C_1210_3225Metric, F.Cu at (79.7, 90.7)
- added C5: 1nF, Capacitor_SMD:C_0603_1608Metric, F.Cu at (108.3, 87.8)
- added C6: 47uF, Capacitor_SMD:C_1210_3225Metric, F.Cu at (111.2, 101.2)
- added C7: 47uF, Capacitor_SMD:C_1210_3225Metric, F.Cu at (111.2, 97.9)
- added C8: 220uF, Capacitor_SMD:CP_Elec_10x10.5, F.Cu at (103.0, 81.0)
- added C9: 10n, Capacitor_SMD:C_0805_2012Metric, F.Cu at (88.0, 91.2)
- added D1: 1N4148, Diode_SMD:D_SOD-323, F.Cu at (87.1, 101.0)
- added D2: SBR8U60P5-7, Diode_SMD:D_PowerDI-5, F.Cu at (111.6, 92.4)
- added D3: BAV21, Diode_SMD:D_SOD-323_HandSoldering, F.Cu at (87.0, 94.0)
- added J1: 013_PoE_rectified, on_edge:on_edge_2x05_device, F.Cu at (77.0, 80.6)
- added J2: 003_power, on_edge:on_edge_2x05_host, F.Cu at (114.0, 80.5)
- added R1: 5.1k, Resistor_SMD:R_0603_1608Metric, F.Cu at (87.2, 97.8)
- added R2: 20k, Resistor_SMD:R_0603_1608Metric, F.Cu at (84.6, 101.5)
- added R3: 41.2R, Resistor_SMD:R_0603_1608Metric, F.Cu at (78.0, 94.7)
- added R4: 24.9k, Resistor_SMD:R_0603_1608Metric, F.Cu at (80.3, 100.2)
- added R5: 49.9k, Resistor_SMD:R_0603_1608Metric, F.Cu at (84.6, 100.0)
- added R6: 110k, Resistor_SMD:R_0603_1608Metric, F.Cu at (82.3, 100.8)
- added R7: 20R, Resistor_SMD:R_0603_1608Metric, F.Cu at (111.3, 87.8)
- added R8: 10K, Resistor_SMD:R_1206_3216Metric, F.Cu at (85.8, 90.7)
- added U1: MP8007, Package_DFN_QFN:QFN-28-1EP_4x5mm_P0.5mm_EP2.65x3.65mm_ThermalVias, F.Cu at (81.8, 96.0)
- added U2: POE13P-50L, b075:Transformer_Coilcraft_POE13P, F.Cu at (99.0, 95.0)
Routing:
- net /flyback/PoE+: track 0.00 -> 78.2 mm, vias 0 -> 10
- net /5V: track 0.00 -> 75.3 mm, vias 0 -> 6
- net /flyback/GNDPWR: track 0.00 -> 51.6 mm, vias 0 -> 11
- net GND: track 0.00 -> 37.2 mm, vias 0 -> 39
- net /flyback/PoE-: track 0.00 -> 32.4 mm, vias 0 -> 8
- net /3.3V: track 0.00 -> 32.2 mm
- net /flyback/transformer_out: track 0.00 -> 14.8 mm
- net Net-(D1-Pad2): track 0.00 -> 14.2 mm
- net /flyback/SW: track 0.00 -> 11.9 mm
- net /flyback/FB1: track 0.00 -> 4.46 mm
- net Net-(C9-Pad2): track 0.00 -> 4.01 mm
- net /flyback/VCC: track 0.00 -> 3.05 mm
- net Net-(R5-Pad1): track 0.00 -> 2.13 mm
- net Net-(R3-Pad1): track 0.00 -> 1.77 mm
- net Net-(R4-Pad2): track 0.00 -> 1.47 mm
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- added copper zone on B.Cu, net /5V
- added copper zone on F.Cu, net /5V
- added copper zone on B.Cu, net /flyback/GNDPWR
- added copper zone on F.Cu, net /flyback/GNDPWR
- added copper zone on F.Cu, net /flyback/PoE+
- added copper zone on F.Cu, net /flyback/PoE-
- added copper zone on F.Cu, net /flyback/SW
- added copper zone on F.Cu, net /flyback/transformer_out
- added copper zone on B.Cu, net GND
- added copper zone on F.Cu, net GND
Other:
- board size 21 x 13 mm -> 37 x 29 mm
- rule pad_to_mask_clearance: 0 -> 0.04
- board text added: "osf.003"
- board text added: "osf.013"
- board text added: "osf.b075.v1.0"
